Commit message: remove definition of pi as it already predefined

File: tams_motorhand_description/urdf/biotac.urdf.xacro (robot description, xacro)
@@ -1,5 +1,4 @@
 <?xml version="1.0"?>
 <robot xmlns:xacro="http://www.ros.org/wiki/xacro" name="biotac_links">
-  <xacro:property name="pi" value="3.1415926535897931" />
   <xacro:macro name="biotac" params="prefix">
     <link name="${prefix}ff_biotac_link">
