Commit message: generalize description to support both motorhands
"left=true" now uses the description for the new left motorhand with PST sensors

File: tams_motorhand_description/urdf/tams_motorhand.urdf.xacro (robot description, xacro)
@@ -5,8 +5,14 @@
   <xacro:include filename="$(find sr_description)/other/xacro/gazebo/gazebo.urdf.xacro" />
   <xacro:include filename="$(find tams_motorhand_description)/urdf/biotac.urdf.xacro" />
-  <xacro:macro name="tams_motorhand" params="prefix">
-    <!-- shadow motorhand BioTac -->
-    <xacro:shadowhand muscletrans="false" muscle="false" bio="true" bt_sp="false" ubi="false" eli="false" reflect="1.0" prefix="${prefix}" lf="true" />
-    <xacro:biotac prefix="${prefix}" />
+  <xacro:macro name="tams_motorhand" params="prefix left:=false">
+    <xacro:unless value="${left}">
+      <!-- shadow motorhand BioTac -->
+      <xacro:shadowhand muscletrans="false" muscle="false" bio="true" bt_sp="false" ubi="false" eli="false" reflect="1.0" prefix="${prefix}" lf="true" />
+      <xacro:biotac prefix="${prefix}" />
+    </xacro:unless>
+    <xacro:if value="${left}">
+      <!-- shadow motorhand BioTac -->
+      <xacro:shadowhand muscletrans="false" muscle="false" bio="false" bt_sp="false" ubi="false" eli="false" reflect="-1.0" prefix="${prefix}" lf="true" />
+    </xacro:if>
   </xacro:macro>
 </robot>

Commit message: modify tams shadow hands according to upstream change, need to use sr_common noetic version

File: tams_motorhand_description/urdf/tams_motorhand.urdf.xacro (robot description, xacro)
@@ -2,16 +2,14 @@
 <robot xmlns:xacro="http://www.ros.org/wiki/xacro" name="tams_motorhand" >
   <!-- include macro definitions -->
-  <xacro:include filename="$(find sr_description)/hand/xacro/full_hand.urdf.xacro" />
-  <xacro:include filename="$(find sr_description)/other/xacro/gazebo/gazebo.urdf.xacro" />
-  <xacro:macro name="tams_motorhand" params="prefix type">
+  <xacro:include filename="$(find sr_description)/hand/xacro/hand.urdf.xacro" />
+  <xacro:include filename="$(find sr_description)/other/xacro/gazebo.urdf.xacro" />
+  <xacro:macro name="tams_motorhand" params="type">
     <xacro:if value="${type == 'right_biotac'}">
       <!-- shadow motorhand BioTac -->
-      <xacro:shadowhand muscletrans="false" muscle="false" bio="true" bt_sp="false" ubi="false" eli="false" reflect="1.0" prefix="${prefix}" lf="true" />
-      <xacro:include filename="$(find tams_motorhand_description)/urdf/biotac.urdf.xacro" />
-      <xacro:biotac prefix="${prefix}" />
+      <xacro:sr_hand hand_type="hand_e" hand_version="E3M5" side="right" fingers="all" tip_sensors="bt_2p" prox_sensors="none" mid_sensors="none" palm_sensor="none" />
     </xacro:if>
     <xacro:if value="${type == 'left_pst'}">
       <!-- shadow left motorhand PST sensing -->
-      <xacro:shadowhand muscletrans="false" muscle="false" bio="false" bt_sp="false" ubi="false" eli="false" reflect="-1.0" prefix="${prefix}" lf="true" />
+      <xacro:sr_hand hand_type="hand_e" hand_version="E3M5" side="left" fingers="all" tip_sensors="pst" prox_sensors="none" mid_sensors="none" palm_sensor="none" />
     </xacro:if>
   </xacro:macro>
