Commit message: generalize repository layout to support new left hand as well
- generalize xacro macro
- provide a generic tams_motorhand_standalone.urdf.xacro as a robot file with a mandatory 'type' parameter
- add right_biotac_hand_ prefix to all specific launch files
- generalize stub to support both hands

Trixi's launch files will have to be adapted to these changes. (Sorry to whoever reads this, it's best done when you
actually can run the launch files in the contexts they should be executed in).

File: tams_motorhand_description/robots/tams_motorhand_standalone.urdf.xacro (robot description, xacro)
@@ -7,11 +7,12 @@
   <xacro:include filename="$(find tams_motorhand_description)/urdf/tams_motorhand.urdf.xacro" />
   <xacro:include filename="$(find sr_description)/materials.urdf.xacro" />
-  <!-- hand with cylindrical base drifts in gazebo, attach it to the world -->
-  <link name="world" />
-  <joint name="rh_world_joint" type="fixed">
-    <parent link="world" />
-    <child link="rh_forearm" />
-    <origin xyz="0.0 0.0 0.0" rpy="0.0 0.0 0.0" />
-  </joint>
-  <xacro:tams_motorhand prefix="rh_" type="right_biotac" />
+  <!--
+       In this robot description the shadow hand is not attached to a parent link.
+       This description is isolated from the rest of the robot and used only by the shadow-modules.
+       ros_control tries to load all joints/transmissions it can find in the robot_description,
+       so we feed it only the shadow hand here.
+       - v4hn@20200830
+  -->
+  <xacro:arg name="type" />
+  <xacro:tams_motorhand prefix="lh_" type="$(arg type)" />
 </robot>

File: tams_motorhand_description/urdf/tams_motorhand.urdf.xacro (robot description, xacro)
@@ -4,13 +4,13 @@
   <xacro:include filename="$(find sr_description)/hand/xacro/full_hand.urdf.xacro" />
   <xacro:include filename="$(find sr_description)/other/xacro/gazebo/gazebo.urdf.xacro" />
-  <xacro:include filename="$(find tams_motorhand_description)/urdf/biotac.urdf.xacro" />
-  <xacro:macro name="tams_motorhand" params="prefix left:=false">
-    <xacro:unless value="${left}">
+  <xacro:macro name="tams_motorhand" params="prefix type">
+    <xacro:if value="${type == 'right_biotac'}">
       <!-- shadow motorhand BioTac -->
       <xacro:shadowhand muscletrans="false" muscle="false" bio="true" bt_sp="false" ubi="false" eli="false" reflect="1.0" prefix="${prefix}" lf="true" />
+      <xacro:include filename="$(find tams_motorhand_description)/urdf/biotac.urdf.xacro" />
       <xacro:biotac prefix="${prefix}" />
-    </xacro:unless>
-    <xacro:if value="${left}">
-      <!-- shadow motorhand BioTac -->
+    </xacro:if>
+    <xacro:if value="${type == 'left_pst'}">
+      <!-- shadow left motorhand PST sensing -->
       <xacro:shadowhand muscletrans="false" muscle="false" bio="false" bt_sp="false" ubi="false" eli="false" reflect="-1.0" prefix="${prefix}" lf="true" />
     </xacro:if>
